Commit message: chore

File: urdf/cibo.urdf (robot description, URDF)
Before this commit: robot cibo, 7 links, 6 joints
Links:
- removed link camera_01_link
- removed link camera_02_link
- added link front_camera_link; visual box size=0.0123 0.0653 0.0225
- added link top_camera_link; visual box size=0.0123 0.0653 0.0225
Joints:
- removed joint camera_01_joint
- removed joint camera_02_joint
- added joint front_camera_joint: type fixed, parent vertical_bar_link, child front_camera_link, origin xyz=0.16 0.0 -0.311 rpy=0 0 0
- added joint top_camera_joint: type fixed, parent horizontal_bar_link, child top_camera_link, origin xyz=0.025 0.0 0.2 rpy=-3.14 0 0

Commit message: chore

File: urdf/cibo.urdf (robot description, URDF)
Before this commit: robot cibo, 7 links, 6 joints
Joints:
- joint front_camera_joint: origin xyz=0.16 0.0 -0.311 rpy=0 0 0 -> xyz=0.16 0.0 -0.106 rpy=0 0 0

Commit message: chore:

File: urdf/cibo.urdf (robot description, URDF)
Before this commit: robot cibo, 7 links, 6 joints
Joints:
- joint top_camera_joint: origin xyz=0.025 0.0 0.2 rpy=-3.14 0 0 -> xyz=0.025 0.0 0.28 rpy=-3.14 0 0
